Commit message: Fixed controller spawning

File: car_assembly/urdf/oldcar_assembly.urdf (robot description, URDF)
Before this commit: robot car_assembly, 8 links, 7 joints
Links:
- removed link dummy_link
- link back_left_wheel_link: mass 0.929515950960187 -> 0.92951595082452
- link back_right_wheel_link: mass 0.929515950263186 -> 0.929515950065346
- link front_left_steer_link: mass 0.979289571979995 -> 0.979289581300228
- link front_left_wheel_link: mass 0.929515950852005 -> 0.929515950960186
- link front_right_steer_link: mass 0.979289566987531 -> 0.9792895843257
- link front_right_wheel_link: mass 0.929515949350559 -> 0.92951595459559
Joints:
- removed joint dummy_joint
- joint back_left_wheel_joint: origin xyz=0.32894 -0.11589 -0.017794 rpy=-1.5708 1.4356 -3.1208 -> xyz=0.328921249974496 -0.114964083839878 -0.0177944693206667 rpy=-1.5707963267949 0.469083696110007 -3.12082450627461
- joint back_right_wheel_joint: origin xyz=0.32174 0.23067 -0.017794 rpy=1.5708 0 -3.1208 -> xyz=0.321763483964631 0.229637520986015 -0.0177944693206667 rpy=1.5707963267949 -0.291614530450468 -3.12082450627461
- joint front_left_steer_joint: origin xyz=-0.17971 -0.089917 0 rpy=1.5708 0 0.019283 -> xyz=-0.17971 -0.089917 0 rpy=1.5708 0 0.094044; type continuous -> revolute
- joint front_left_wheel_joint: origin xyz=0.00012521 -0.017794 0.035923 rpy=0 0 1.0465 -> xyz=0.000125211657348218 -0.0177944693206653 0.014651735605834 rpy=0 0 -2.49079241735017
- joint front_right_steer_joint: origin xyz=-0.18538 0.18307 0 rpy=1.5708 0 3.1278 -> xyz=-0.18538 0.18307 0 rpy=1.5708 0 3.1235; type continuous -> revolute
- joint front_right_wheel_joint: origin xyz=0.00012521 -0.017794 0.04129 rpy=0 0 -0.43105 -> xyz=0.000125211657348301 -0.0177944693206666 0.0412999511488255 rpy=0 0 -0.431045729807837
