Commit message: Adding ROS package for car assembly

File: car_assembly/urdf/car_assembly.urdf.xacro (robot description, xacro)
@@ -1,8 +1,9 @@
-<?xml version="1.0" encoding="utf-8"?>
+<?xml version="1.0" ?>
 <!-- This URDF was automatically created by SolidWorks to URDF Exporter! Originally created by Stephen Brawner (brawner@gmail.com)
      Commit Version: 1.6.0-4-g7f85cfe  Build Version: 1.6.7995.38578
      For more information, please see http://wiki.ros.org/sw_urdf_exporter -->
-<robot
-  name="car_assembly">
+<robot name="car_assembly" xmlns:xacro="http://ros.org/wiki/xacro">
+  <!-- # Add this be  fore base link -->
+  <link name="dummy_link"></link>
   <link
     name="base_link">
@@ -45,4 +46,10 @@
     </collision>
   </link>
+  <!-- # Add this after base link -->
+  <joint name="dummy_joint" type="fixed">
+      <origin rpy="0 0 0" xyz="0 0 0" />
+      <parent link="dummy_link"/>
+      <child link="base_link"/>
+  </joint>
   <link
     name="back_left_wheel_link">
@@ -263,5 +270,5 @@
   </joint>
   <link
-    name="front_right_steer_joint">
+    name="front_right_steer_link">
     <inertial>
       <origin
@@ -284,5 +291,5 @@
       <geometry>
         <mesh
-          filename="package://car_assembly/meshes/front_right_steer_joint.STL" />
+          filename="package://car_assembly/meshes/front_right_steer_link.STL" />
       </geometry>
       <material
@@ -298,5 +305,5 @@
       <geometry>
         <mesh
-          filename="package://car_assembly/meshes/front_right_steer_joint.STL" />
+          filename="package://car_assembly/meshes/front_right_steer_link.STL" />
       </geometry>
     </collision>
@@ -311,5 +318,5 @@
       link="base_link" />
     <child
-      link="front_right_steer_joint" />
+      link="front_right_steer_link" />
     <axis
       xyz="0 1 0" />
@@ -367,5 +374,5 @@
       rpy="0 0 -0.43105" />
     <parent
-      link="front_right_steer_joint" />
+      link="front_right_steer_link" />
     <child
       link="front_right_wheel_link" />
@@ -373,3 +380,16 @@
       xyz="0 0 1" />
   </joint>
+  <!-- <xacro:macro name="body_color">
+    <visual>
+    <material>
+        <ambient>0.8 0.558823529411765 0.1 1</ambient>
+        <diffuse>0.8 0.558823529411765 0.1 1</diffuse>
+        <specular>0.1 0.1 0.1 1</specular>
+        <emissive>0 0 0 0</emissive>
+    </material>
+    </visual>
+  </xacro:macro>
+  <gazebo reference="base_link">
+    <xacro:body_color />
+  </gazebo> -->
 </robot>

Commit message: Added code for proportional velocity controller

File: car_assembly/urdf/car_assembly.urdf.xacro (robot description, xacro)
@@ -210,6 +210,6 @@
       xyz="0 1 0" />
     <limit
-      lower="-0.785"
-      upper="0.785"
+      lower="-1.571"
+      upper="1.571"
       effort="100"
       velocity="3.14" />
@@ -321,6 +321,6 @@
       xyz="0 1 0" />
     <limit
-      lower="-0.785"
-      upper="0.785"
+      lower="-1.571"
+      upper="1.571"
       effort="100"
       velocity="3.14" />
@@ -379,4 +379,97 @@
       xyz="0 0 1" />
   </joint>
+  <!-- Lidar definition -->
+  <link name="lidar_link">
+   <inertial>
+     <origin xyz="0 0 0" rpy="0 0 0"/>
+     <mass value="1"/>
+     <inertia ixx="100"  ixy="0"  ixz="0" iyy="100" iyz="0" izz="100" />
+   </inertial>
+   <visual>
+     <origin xyz="0 0 0" rpy="0 0 0" />
+     <geometry>
+       <cylinder radius="0.1524" length="0.1"/>
+     </geometry>
+     <material name="Cyan">
+       <color rgba="0 1.0 1.0 1.0"/>
+     </material>
+   </visual>
+   <collision>
+     <origin xyz="0 0 0" rpy="0 0 0"/>
+     <geometry>
+       <cylinder radius="0.1524" length="0.1"/>
+     </geometry>
+   </collision>
+ </link>
+ <joint
+    name="lidar_joint"
+    type="fixed">
+    <origin
+      xyz="0.0686 0.04735 0.3048"
+      rpy="0 0 0" />
+    <parent
+      link="base_link" />
+    <child
+      link="lidar_link" />
+    <axis
+      xyz="0 0 1" />
+  </joint>
+  <gazebo reference="lidar_link">
+    <sensor name="lidar" type="ray">
+      <pose>0.0 0.0 0.0 0 0 0</pose>
+      <always_on>true</always_on>
+      <visualize>false</visualize>
+      <update_rate>5</update_rate>
+      <ray>
+        <scan>
+          <horizontal>
+            <samples>360</samples>
+            <resolution>1.00000</resolution>
+            <min_angle>0.000000</min_angle>
+            <max_angle>6.280000</max_angle>
+          </horizontal>
+        </scan>
+        <range>
+          <min>0.16</min>
+          <max>3.5</max>
+          <resolution>0.015000</resolution>
+        </range>
+        <noise>
+          <type>gaussian</type>
+          <mean>0.0</mean>
+          <stddev>0.01</stddev>
+        </noise>
+      </ray>
+      <plugin name="scan" filename="libgazebo_ros_ray_sensor.so">
+        <ros>
+          <remapping>~/out:=scan</remapping>
+        </ros>
+        <output_type>sensor_msgs/LaserScan</output_type>
+        <frame_name>lidar_link</frame_name>
+      </plugin>
+    </sensor>
+  </gazebo>
+  <!-- IMU -->
+  <gazebo reference="base_link">
+    <gravity>true</gravity>
+    <sensor name="imu_sensor" type="imu">
+      <always_on>true</always_on>
+      <update_rate>100</update_rate>
+      <visualize>true</visualize>
+      <topic>__default_topic__</topic>
+      <plugin filename="libgazebo_ros_imu_sensor.so" name="imu_plugin">
+        <topicName>imu</topicName>
+        <bodyName>base_link</bodyName>
+        <updateRateHZ>10.0</updateRateHZ>
+        <gaussianNoise>0.0</gaussianNoise>
+        <xyzOffset>0 0 0</xyzOffset>
+        <rpyOffset>0 0 0</rpyOffset>
+        <frameName>base_link</frameName>
+        <initialOrientationAsReference>false</initialOrientationAsReference>
+      </plugin>
+      <pose>0 0 0 0 0 0</pose>
+    </sensor>
+  </gazebo>
+  <!-- ROS Gazebo controls -->
   <ros2_control name="GazeboSystem" type="system">
     <hardware>
@@ -421,6 +514,6 @@
     <joint name="front_left_steer_joint">
         <command_interface name="position">
-            <param name="min">-0.785</param>
-            <param name="max">0.785</param>
+            <param name="min">-1.571</param>
+            <param name="max">1.571</param>
         </command_interface>
         <state_interface name="position"/>
@@ -429,6 +522,6 @@
     <joint name="front_right_steer_joint">
         <command_interface name="position">
-            <param name="min">-0.785</param>
-            <param name="max">0.785</param>
+            <param name="min">-1.571</param>
+            <param name="max">1.571</param>
         </command_interface>
         <state_interface name="position"/>

Commit message: Updated model to remove slight yaw in front steer wheel

File: car_assembly/urdf/car_assembly.urdf.xacro (robot description, xacro)
@@ -10,15 +10,15 @@
     <inertial>
       <origin
-        xyz="0.0984933879187388 0.139538868480493 -0.0524164095634679"
-        rpy="0 0 0" />
-      <mass
-        value="42.437819295697" />
-      <inertia
-        ixx="0.793248965062798"
-        ixy="0.12082958397428"
-        ixz="0.0438841068170688"
-        iyy="3.47432493664263"
-        iyz="-0.00250976744462374"
-        izz="2.9050823428007" />
+        xyz="0.098493 0.13954 -0.052416"
+        rpy="0 0 0" />
+      <mass
+        value="43.287" />
+      <inertia
+        ixx="0.80911"
+        ixy="0.12325"
+        ixz="0.044762"
+        iyy="3.5438"
+        iyz="-0.00256"
+        izz="2.9632" />
     </inertial>
     <visual>
@@ -52,18 +52,71 @@
   </joint>
   <link
+    name="back_right_wheel_link">
+    <inertial>
+      <origin
+        xyz="2.191E-11 2.3697E-10 0.047994"
+        rpy="0 0 0" />
+      <mass
+        value="0.92952" />
+      <inertia
+        ixx="0.0033456"
+        ixy="-1.3555E-12"
+        ixz="-4.9134E-13"
+        iyy="0.0033456"
+        iyz="-5.1504E-12"
+        izz="0.0056993" />
+    </inertial>
+    <visual>
+      <origin
+        xyz="0 0 0"
+        rpy="0 0 0" />
+      <geometry>
+        <mesh
+          filename="package://car_assembly/meshes/back_right_wheel_link.STL" />
+      </geometry>
+      <material
+        name="">
+        <color
+          rgba="0.25098 0.25098 0.25098 1" />
+      </material>
+    </visual>
+    <collision>
+      <origin
+        xyz="0 0 0"
+        rpy="0 0 0" />
+      <geometry>
+        <mesh
+          filename="package://car_assembly/meshes/back_right_wheel_link.STL" />
+      </geometry>
+    </collision>
+  </link>
+  <joint
+    name="back_right_wheel_joint"
+    type="continuous">
+    <origin
+      xyz="0.32174 0.23067 -0.017794"
+      rpy="1.5708 0 -3.1208" />
+    <parent
+      link="base_link" />
+    <child
+      link="back_right_wheel_link" />
+    <axis
+      xyz="0 0 1" />
+  </joint>
+  <link
     name="back_left_wheel_link">
     <inertial>
       <origin
-        xyz="2.20701026898418E-11 2.3632068524293E-10 0.0485238176719048"
-        rpy="0 0 0" />
-      <mass
-        value="0.929515950960187" />
-      <inertia
-        ixx="0.00334561969791303"
-        ixy="-1.35412065084509E-12"
-        ixz="-4.94448256074592E-13"
-        iyy="0.00334561968377833"
-        iyz="-5.13307857997287E-12"
-        izz="0.00569925253456415" />
+        xyz="2.207E-11 2.3632E-10 0.048524"
+        rpy="0 0 0" />
+      <mass
+        value="0.92952" />
+      <inertia
+        ixx="0.0033456"
+        ixy="-1.3541E-12"
+        ixz="-4.9445E-13"
+        iyy="0.0033456"
+        iyz="-5.1331E-12"
+        izz="0.0056993" />
     </inertial>
     <visual>
@@ -78,5 +131,5 @@
         name="">
         <color
-          rgba="0.250980392156863 0.250980392156863 0.250980392156863 1" />
+          rgba="0.25098 0.25098 0.25098 1" />
       </material>
     </visual>
@@ -105,53 +158,106 @@
   </joint>
   <link
-    name="back_right_wheel_link">
-    <inertial>
-      <origin
-        xyz="2.19100848575238E-11 2.36971997580326E-10 0.0479937520853098"
-        rpy="0 0 0" />
-      <mass
-        value="0.929515950263186" />
-      <inertia
-        ixx="0.00334561969667993"
-        ixy="-1.35549519578422E-12"
-        ixz="-4.91341972804708E-13"
-        iyy="0.00334561968253039"
-        iyz="-5.15041254599154E-12"
-        izz="0.00569925253266686" />
-    </inertial>
-    <visual>
-      <origin
-        xyz="0 0 0"
-        rpy="0 0 0" />
-      <geometry>
-        <mesh
-          filename="package://car_assembly/meshes/back_right_wheel_link.STL" />
-      </geometry>
-      <material
-        name="">
-        <color
-          rgba="0.250980392156863 0.250980392156863 0.250980392156863 1" />
-      </material>
-    </visual>
-    <collision>
-      <origin
-        xyz="0 0 0"
-        rpy="0 0 0" />
-      <geometry>
-        <mesh
-          filename="package://car_assembly/meshes/back_right_wheel_link.STL" />
+    name="front_right_steer_link">
+    <inertial>
+      <origin
+        xyz="1.6654E-05 0.03399 0.0088169"
+        rpy="0 0 0" />
+      <mass
+        value="0.99888" />
+      <inertia
+        ixx="0.0038487"
+        ixy="8.602E-07"
+        ixz="-9.5628E-07"
+        iyy="0.0012132"
+        iyz="0.00045607"
+        izz="0.0033123" />
+    </inertial>
+    <visual>
+      <origin
+        xyz="0 0 0"
+        rpy="0 0 0" />
+      <geometry>
+        <mesh
+          filename="package://car_assembly/meshes/front_right_steer_link.STL" />
+      </geometry>
+      <material
+        name="">
+        <color
+          rgba="1 1 1 1" />
+      </material>
+    </visual>
+    <collision>
+      <origin
+        xyz="0 0 0"
+        rpy="0 0 0" />
+      <geometry>
+        <mesh
+          filename="package://car_assembly/meshes/front_right_steer_link.STL" />
       </geometry>
     </collision>
   </link>
   <joint
-    name="back_right_wheel_joint"
+    name="front_right_steer_joint"
     type="continuous">
     <origin
-      xyz="0.32174 0.23067 -0.017794"
+      xyz="-0.18538 0.18307 0"
       rpy="1.5708 0 -3.1208" />
     <parent
       link="base_link" />
     <child
-      link="back_right_wheel_link" />
+      link="front_right_steer_link" />
+    <axis
+      xyz="0 1 0" />
+  </joint>
+  <link
+    name="front_right_wheel_link">
+    <inertial>
+      <origin
+        xyz="2.207E-11 2.3632E-10 0.049174"
+        rpy="0 0 0" />
+      <mass
+        value="0.92952" />
+      <inertia
+        ixx="0.0033456"
+        ixy="-1.3541E-12"
+        ixz="-4.9445E-13"
+        iyy="0.0033456"
+        iyz="-5.1331E-12"
+        izz="0.0056993" />
+    </inertial>
+    <visual>
+      <origin
+        xyz="0 0 0"
+        rpy="0 0 0" />
+      <geometry>
+        <mesh
+          filename="package://car_assembly/meshes/front_right_wheel_link.STL" />
+      </geometry>
+      <material
+        name="">
+        <color
+          rgba="0.25098 0.25098 0.25098 1" />
+      </material>
+    </visual>
+    <collision>
+      <origin
+        xyz="0 0 0"
+        rpy="0 0 0" />
+      <geometry>
+        <mesh
+          filename="package://car_assembly/meshes/front_right_wheel_link.STL" />
+      </geometry>
+    </collision>
+  </link>
+  <joint
+    name="front_right_wheel_joint"
+    type="continuous">
+    <origin
+      xyz="0.00012521 -0.017794 0.035876"
+      rpy="0 0 -0.34569" />
+    <parent
+      link="front_right_steer_link" />
+    <child
+      link="front_right_wheel_link" />
     <axis
       xyz="0 0 1" />
@@ -161,15 +267,15 @@
     <inertial>
       <origin
-        xyz="1.66541358932737E-05 0.0339902365470534 0.00881686894273455"
-        rpy="0 0 0" />
-      <mass
-        value="0.979289571979995" />
-      <inertia
-        ixx="0.00377322322154386"
-        ixy="8.43332889853372E-07"
-        ixz="-9.37533254204548E-07"
-        iyy="0.00118944602771482"
-        iyz="0.000447122978840801"
-        izz="0.00324735800237895" />
+        xyz="1.6654E-05 0.03399 0.0088169"
+        rpy="0 0 0" />
+      <mass
+        value="0.99888" />
+      <inertia
+        ixx="0.0038487"
+        ixy="8.602E-07"
+        ixz="-9.5628E-07"
+        iyy="0.0012132"
+        iyz="0.00045607"
+        izz="0.0033123" />
     </inertial>
     <visual>
@@ -202,5 +308,5 @@
     <origin
       xyz="-0.17971 -0.089917 0"
-      rpy="1.5708 0 0.019283" />
+      rpy="1.5708 0 0.020768" />
     <parent
       link="base_link" />
@@ -209,9 +315,4 @@
     <axis
       xyz="0 1 0" />
-    <limit
-      lower="-1.571"
-      upper="1.571"
-      effort="100"
-      velocity="3.14" />
   </joint>
   <link
@@ -219,15 +320,15 @@
     <inertial>
       <origin
-        xyz="2.21104939912564E-11 2.36410446774471E-10 0.0491271368458189"
-        rpy="0 0 0" />
-      <mass
-        value="0.929515950852005" />
-      <inertia
-        ixx="0.00334561969772165"
-        ixy="-1.3543360132468E-12"
-        ixz="-4.955219516504E-13"
-        iyy="0.00334561968358468"
-        iyz="-5.13540815097078E-12"
-        izz="0.00569925253426966" />
+        xyz="2.207E-11 2.3632E-10 0.049539"
+        rpy="0 0 0" />
+      <mass
+        value="0.92952" />
+      <inertia
+        ixx="0.0033456"
+        ixy="-1.3541E-12"
+        ixz="-4.9445E-13"
+        iyy="0.0033456"
+        iyz="-5.1331E-12"
+        izz="0.0056993" />
     </inertial>
     <visual>
@@ -242,5 +343,5 @@
         name="">
         <color
-          rgba="0.250980392156863 0.250980392156863 0.250980392156863 1" />
+          rgba="0.25098 0.25098 0.25098 1" />
       </material>
     </visual>
@@ -259,5 +360,5 @@
     type="continuous">
     <origin
-      xyz="0.00012521 -0.017794 0.035923"
+      xyz="0.00012521 -0.017794 0.035511"
       rpy="0 0 1.0465" />
     <parent
@@ -265,115 +366,4 @@
     <child
       link="front_left_wheel_link" />
-    <axis
-      xyz="0 0 1" />
-  </joint>
-  <link
-    name="front_right_steer_link">
-    <inertial>
-      <origin
-        xyz="1.66538436364716E-05 0.0339902362547982 0.00881686876318738"
-        rpy="0 0 0" />
-      <mass
-        value="0.979289566987531" />
-      <inertia
-        ixx="0.00377322320424715"
-        ixy="8.43350650471856E-07"
-        ixz="-9.37529907092586E-07"
-        iyy="0.00118944602573503"
-        iyz="0.000447122989383998"
-        izz="0.00324735798453781" />
-    </inertial>
-    <visual>
-      <origin
-        xyz="0 0 0"
-        rpy="0 0 0" />
-      <geometry>
-        <mesh
-          filename="package://car_assembly/meshes/front_right_steer_link.STL" />
-      </geometry>
-      <material
-        name="">
-        <color
-          rgba="1 1 1 1" />
-      </material>
-    </visual>
-    <collision>
-      <origin
-        xyz="0 0 0"
-        rpy="0 0 0" />
-      <geometry>
-        <mesh
-          filename="package://car_assembly/meshes/front_right_steer_link.STL" />
-      </geometry>
-    </collision>
-  </link>
-  <joint
-    name="front_right_steer_joint"
-    type="continuous">
-    <origin
-      xyz="-0.18538 0.18307 0"
-      rpy="1.5708 0 3.1278" />
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