Commit message: Initial code for homework 3 and the diagram for project 2

File: project_1/new_car_assembly_export/urdf/new_car_assembly_export.urdf (robot description, URDF)
Before this commit: robot new_car_assembly_export, 7 links, 6 joints
Links:
- link front_right_steer_link: mass 0.9792895843257 -> 0.979289573985709
- link front_right_wheel_link: mass 0.92951595459559 -> 0.929515950960185
Joints:
- joint back_right_wheel_joint: origin xyz=0.321763483964631 0.229637520986015 -0.0177944693206667 rpy=1.5707963267949 -0.291614530450468 -3.12082450627461 -> xyz=0.32176 0.22964 -0.017794 rpy=1.5708 -0.29161 -3.1208
- joint front_left_steer_joint: origin xyz=-0.17971 -0.089917 0 rpy=1.5708 0 0.094044 -> xyz=-0.179708588418403 -0.0899166088816682 0 rpy=1.5707963267949 0 0.0940442461119153
- joint front_right_steer_joint: origin xyz=-0.18538 0.18307 0 rpy=1.5708 0 3.1235 -> xyz=-0.18538 0.18307 0 rpy=1.5708 0 3.1208
