Commit message: Added front LiDAR

File: aircraft_inspection_robot/urdf/aircraft_inspection_robot.urdf (robot description, URDF)
Before this commit: robot aircraft_inspection_robot, 15 links, 14 joints
Links:
- added link front_lidar_sensor_link
Joints:
- added joint front_lidar_sensor_joint: type fixed, parent front_lidar_link, child front_lidar_sensor_link, origin xyz=0 0.25 0 rpy=1.571 1.571 0

Commit message: Updated front lidar position

File: aircraft_inspection_robot/urdf/aircraft_inspection_robot.urdf (robot description, URDF)
Before this commit: robot aircraft_inspection_robot, 16 links, 15 joints
Joints:
- joint front_lidar_sensor_joint: origin xyz=0 0.25 0 rpy=1.571 1.571 0 -> xyz=0 -0.05 0 rpy=1.571 1.571 0

Commit message: Added rear lidar to aircraft robot

File: aircraft_inspection_robot/urdf/aircraft_inspection_robot.urdf (robot description, URDF)
Before this commit: robot aircraft_inspection_robot, 16 links, 15 joints
Links:
- added link rear_lidar_sensor_link
Joints:
- added joint rear_lidar_sensor_joint: type fixed, parent rear_lidar_link, child rear_lidar_sensor_link, origin xyz=0 -0.05 0 rpy=1.571 1.571 0
