Commit message: Added depth camera

File: aircraft_inspection_robot/urdf/aircraft_inspection_robot.urdf.xacro (robot description, xacro)
@@ -991,4 +991,37 @@
     </sensor>
   </gazebo>
+  <!-- Depth Camera -->
+  <link name="depth_camera_sensor_link"></link>
+  <joint name="depth_camera_sensor_joint" type="fixed">
+    <origin rpy="-1.571 0 0" xyz="0.2 0 0" />
+    <parent link="camera_link"/>
+    <child link="depth_camera_sensor_link"/>
+  </joint>
+  <gazebo reference="depth_camera_sensor_link">
+    <sensor name="depth_camera" type="depth">
+      <camera name="depth_camera">
+        <!-- Camera properties -->
+        <horizontal_fov>1.047</horizontal_fov>
+        <vertical_fov>0.785</vertical_fov>
+        <image>
+          <width>640</width>
+          <height>480</height>
+        </image>
+        <clip>
+          <near>0.1</near>
+          <far>20.0</far>
+        </clip>
+      </camera>
+      <!-- Depth camera Gazebo plugin -->
+      <plugin name="gazebo_ros_depth_camera" filename="libgazebo_ros_camera.so">
+        <alwaysOn>true</alwaysOn>
+        <updateRate>30.0</updateRate>
+        <cameraName>depth</cameraName>
+        <frameName>depth_camera_sensor_link</frameName>
+        <imageTopicName>image_raw</imageTopicName>
+        <cameraInfoTopicName>camera_info</cameraInfoTopicName>
+      </plugin>
+    </sensor>
+  </gazebo>
   <gazebo>
     <plugin filename="libgazebo_ros2_control.so" name="gazebo_ros2_control">

Commit message: Updated urdf and config for new arm

File: aircraft_inspection_robot/urdf/aircraft_inspection_robot.urdf.xacro (robot description, xacro)
@@ -10,15 +10,15 @@
     <inertial>
       <origin
-        xyz="-0.409737523113878 0.248339713620131 0.209639401630241"
-        rpy="0 0 0" />
-      <mass
-        value="52.4458402259021" />
-      <inertia
-        ixx="1.61796946709653"
-        ixy="-4.26019586297761E-05"
-        ixz="5.36565329733604E-05"
-        iyy="3.60901877519089"
-        iyz="0.00014045219036093"
-        izz="4.89191044456781" />
+        xyz="-0.40974645535857 0.24834344494391 0.242010590101945"
+        rpy="0 0 0" />
+      <mass
+        value="52.3239752391313" />
+      <inertia
+        ixx="0.952539519630922"
+        ixy="-4.26200364814785E-05"
+        ixz="5.36575380324012E-05"
+        iyy="3.80199276879049"
+        iyz="2.4370448304257E-05"
+        izz="4.07464899613958" />
     </inertial>
     <visual>
@@ -33,5 +33,5 @@
         name="">
         <color
-          rgba="1 1 1 1" />
+          rgba="0.250980392156863 0.250980392156863 0.250980392156863 1" />
       </material>
     </visual>
@@ -55,15 +55,15 @@
     <inertial>
       <origin
-        xyz="-0.00725498730999624 -0.159524096445023 -5.18934305249186E-08"
-        rpy="0 0 0" />
-      <mass
-        value="21.0173459101461" />
-      <inertia
-        ixx="0.360630213819554"
-        ixy="-0.0108096413980878"
-        ixz="4.79803425565932E-08"
-        iyy="0.186912416456727"
-        iyz="-2.37737605206146E-07"
-        izz="0.361463047566562" />
+        xyz="-0.00725496120108809 -0.159524101399661 -5.98196165102483E-08"
+        rpy="0 0 0" />
+      <mass
+        value="2.62716823876827" />
+      <inertia
+        ixx="0.0112696941818608"
+        ixy="-0.00033780129369249"
+        ixz="1.4993857049244E-09"
+        iyy="0.00584101301427301"
+        iyz="-7.42930015937879E-09"
+        izz="0.0112957202364551" />
     </inertial>
     <visual>
@@ -95,5 +95,5 @@
     type="fixed">
     <origin
-      xyz="0.308106449560569 0.248338347564378 0.236097315694741"
+      xyz="0.252189298222892 0.248326110601867 0.129347762825463"
       rpy="-1.57091123434865 0 0" />
     <parent
@@ -108,15 +108,15 @@
     <inertial>
       <origin
-        xyz="-0.00725498516150735 0.1695240965549 -5.18932890547497E-08"
-        rpy="0 0 0" />
-      <mass
-        value="21.0173459127111" />
-      <inertia
-        ixx="0.360630214140233"
-        ixy="-0.0108096390967668"
-        ixz="4.79968519505956E-08"
-        iyy="0.18691241620145"
-        iyz="-2.37742872890824E-07"
-        izz="0.361463047569039" />
+        xyz="-0.00725495907227769 -0.159524101502578 -5.98195511736233E-08"
+        rpy="0 0 0" />
+      <mass
+        value="2.62716823908889" />
+      <inertia
+        ixx="0.0112696941918823"
+        ixy="-0.000337801221774006"
+        ixz="1.49990162575632E-09"
+        iyy="0.00584101300629532"
+        iyz="-7.42946478333022E-09"
+        izz="0.0112957202365325" />
     </inertial>
     <visual>
@@ -148,5 +148,5 @@
     type="fixed">
     <origin
-      xyz="0.308106449560569 0.248338347564378 0.236097315694741"
+      xyz="-1.07167463581468 0.248325943235427 0.129347754093208"
       rpy="-1.57068141924114 0 3.14159265358979" />
     <parent
@@ -161,15 +161,15 @@
     <inertial>
       <origin
-        xyz="-5.59829960167235E-14 1.71109293400917E-10 0.103131389958602"
-        rpy="0 0 0" />
-      <mass
-        value="17.0942965183764" />
-      <inertia
-        ixx="0.267032855143768"
-        ixy="-1.12643384679206E-12"
-        ixz="-5.64889032158929E-10"
-        iyy="0.267032853623031"
-        iyz="9.3846801464399E-12"
-        izz="0.388719266107455" />
+        xyz="7.69611511519663E-07 -1.70468712881733E-07 0.102621158507274"
+        rpy="0 0 0" />
+      <mass
+        value="26.0461976105726" />
+      <inertia
+        ixx="0.285954065616882"
+        ixy="7.95282541629767E-07"
+        ixz="1.27020782265502E-07"
+        iyy="0.28595474175216"
+        iyz="-3.78487432157488E-07"
+        izz="0.40415282922357" />
     </inertial>
     <visual>
@@ -184,5 +184,5 @@
         name="">
         <color
-          rgba="0.250980392156863 0.250980392156863 0.250980392156863 1" />
+          rgba="0.792156862745098 0.819607843137255 0.933333333333333 1" />
       </material>
     </visual>
@@ -201,6 +201,6 @@
     type="continuous">
     <origin
-      xyz="-0.117597527934808 -0.0373548329643068 0.101609117592568"
-      rpy="-1.57057710899586 -1.01905526588804 3.14140604048142" />
+      xyz="-0.117597527933808 -0.0373680425515616 0.10160911911045"
+      rpy="-1.57068160265985 -0.0571716575997457 3.14159265358979" />
     <parent
       link="base_link" />
@@ -208,5 +208,5 @@
       link="front_right_wheel_link" />
     <axis
-      xyz="0 0 1" />
+      xyz="0 0 0.999999999978938" />
   </joint>
   <link
@@ -214,15 +214,15 @@
     <inertial>
       <origin
-        xyz="-6.06656651996884E-14 1.71113873070894E-10 -0.10313316315041"
-        rpy="0 0 0" />
-      <mass
-        value="17.0942965183763" />
-      <inertia
-        ixx="0.267032855143761"
-        ixy="-1.14495324383746E-12"
-        ixz="5.64901635417955E-10"
-        iyy="0.267032853623031"
-        iyz="-9.36914437972927E-12"
-        izz="0.388719266107462" />
+        xyz="1.06668829737838E-07 -1.81805510673927E-07 -0.674003005040707"
+        rpy="0 0 0" />
+      <mass
+        value="26.0463242126014" />
+      <inertia
+        ixx="0.285954618303477"
+        ixy="7.68759858498613E-07"
+        ixz="6.28786224972317E-07"
+        iyy="0.285955290913927"
+        iyz="3.7011482934088E-07"
+        izz="0.404153186322765" />
     </inertial>
     <visual>
@@ -237,5 +237,5 @@
         name="">
         <color
-          rgba="0.250980392156863 0.250980392156863 0.250980392156863 1" />
+          rgba="0.792156862745098 0.819607843137255 0.933333333333333 1" />
       </material>
     </visual>
@@ -254,6 +254,6 @@
     type="continuous">
     <origin
-      xyz="-0.117597571165592 0.533998775516627 0.101543464746798"
-      rpy="1.57061905476483 -0.865579426080518 0.00013506316993608" />
+      xyz="-0.117597527933808 -0.0373680425515616 0.10160911911045"
+      rpy="1.57056878031369 -1.04143176730992 0.000196477434083904" />
     <parent
       link="base_link" />
@@ -267,15 +267,15 @@
     <inertial>
       <origin
-        xyz="-6.03961325396085E-14 1.71112679581142E-10 0.103133072201983"
-        rpy="0 0 0" />
-      <mass
-        value="17.0942965183763" />
-      <inertia
-        ixx="0.267032855143761"
-        ixy="-1.14615484325525E-12"
-        ixz="-5.64900110911116E-10"
-        iyy="0.267032853623031"
-        iyz="9.36830792283539E-12"
-        izz="0.388719266107461" />
+        xyz="8.41577684762562E-08 -1.68242609732694E-07 0.102641039115083"
+        rpy="0 0 0" />
+      <mass
+        value="26.0462008072991" />
+      <inertia
+        ixx="0.285954040177974"
+        ixy="7.90067012358279E-07"
+        ixz="-6.50671063736261E-07"
+        iyy="0.285954742544619"
+        iyz="-3.69738156013685E-07"
+        izz="0.40415280236699" />
     </inertial>
     <visual>
@@ -290,5 +290,5 @@
         name="">
         <color
-          rgba="0.250980392156863 0.250980392156863 0.250980392156863 1" />
+          rgba="0.792156862745098 0.819607843137255 0.933333333333333 1" />
       </material>
     </visual>
@@ -307,6 +307,6 @@
     type="continuous">
     <origin
-      xyz="-0.7018 -0.037353 0.10161"
-      rpy="1.5706 -0.87958 0.00013896" />
+      xyz="-0.701797527935311 -0.0373482051170577 0.101609112969085"
+      rpy="1.57064724689163 -0.690734458596981 9.50549862212618E-05" />
     <parent
       link="base_link" />
@@ -320,15 +320,15 @@
     <inertial>
       <origin
-        xyz="-5.65658631046517E-14 1.71111347313513E-10 -0.103131061396203"
-        rpy="0 0 0" />
-      <mass
-        value="17.0942965183761" />
-      <inertia
-        ixx="0.267032855143766"
-        ixy="-1.12798336645332E-12"
-        ixz="5.64892007313028E-10"
-        iyy="0.267032853623031"
-        iyz="-9.37929468555027E-12"
-        izz="0.388719266107457" />
+        xyz="1.29034836829356E-07 -2.66555836092586E-06 -0.673983123389094"
+        rpy="0 0 0" />
+      <mass
+        value="26.0463122941313" />
+      <inertia
+        ixx="0.285954575528675"
+        ixy="7.71478869336928E-07"
+        ixz="6.45837128179966E-07"
+        iyy="0.285955250948586"
+        iyz="7.90647100387111E-07"
+        izz="0.404153156835058" />
     </inertial>
     <visual>
@@ -343,5 +343,5 @@
         name="">
         <color
-          rgba="0.250980392156863 0.250980392156863 0.250980392156863 1" />
+          rgba="0.792156862745098 0.819607843137255 0.933333333333333 1" />
       </material>
     </visual>
@@ -360,6 +360,6 @@
     type="continuous">
     <origin
-      xyz="-0.7018 0.534 0.10154"
-      rpy="-1.5706 -1.0375 3.1414" />
+      xyz="-0.701797527935311 -0.0373482051170577 0.101609112969085"
+      rpy="1.56727528936655 -1.5381898923507 0.00352290998991109" />
     <parent
       link="base_link" />
@@ -367,58 +367,5 @@
       link="back_left_wheel_link" />
     <axis
-      xyz="0 0 1" />
-  </joint>
-  <link
-    name="arm_connector_link">
-    <inertial>
-      <origin
-        xyz="-1.43143330522122E-10 0.0216537321612436 1.10744746706359E-14"
-        rpy="0 0 0" />
-      <mass
-        value="2.62877306618386" />
-      <inertia
-        ixx="0.0207836884851897"
-        ixy="-1.25135931667707E-10"
-        ixz="-2.20944162334301E-25"
-        iyy="0.039713380262994"
-        iyz="-2.37404276874067E-17"
-        izz="0.0207836884851897" />
-    </inertial>
-    <visual>
-      <origin
-        xyz="0 0 0"
-        rpy="0 0 0" />
-      <geometry>
-        <mesh
-          filename="package://aircraft_inspection_robot/meshes/arm_connector_link.STL" />
-      </geometry>
-      <material
-        name="">
-        <color
-          rgba="0.250980392156863 0.250980392156863 0.250980392156863 1" />
-      </material>
-    </visual>
-    <collision>
-      <origin
-        xyz="0 0 0"
-        rpy="0 0 0" />
-      <geometry>
-        <mesh
-          filename="package://aircraft_inspection_robot/meshes/arm_connector_link.STL" />
-      </geometry>
-    </collision>
-  </link>
-  <joint
-    name="arm_connect_joint"
-    type="fixed">
-    <origin
-      xyz="-0.4097 0.24836 0.41908"
-      rpy="1.5707 0 0" />
-    <parent
-      link="base_link" />
-    <child
-      link="arm_connector_link" />
-    <axis
-      xyz="0 0 0" />
+      xyz="0 0 0.999999999993264" />
   </joint>
   <link
@@ -426,15 +373,15 @@
     <inertial>
       <origin
-        xyz="8.98447982677908E-14 0.118624566442621 -7.84175280266197E-10"
-        rpy="0 0 0" />
-      <mass
-        value="16.2102374081522" />
-      <inertia
-        ixx="0.278054099642839"
-        ixy="-4.40146949106952E-14"
-        ixz="1.13856898220502E-16"
-        iyy="0.226366310502593"
-        iyz="6.241749681372E-10"
-        izz="0.320787148766728" />
+        xyz="-1.64295967997052E-07 0.231013183516839 0.049503043395059"
+        rpy="0 0 0" />
+      <mass
+        value="49.4633477448353" />
+      <inertia
+        ixx="1.41939380135235"
+        ixy="-8.90881223634171E-07"
+        ixz="9.56220690256119E-07"
+        iyy="1.27036787158441"
+        iyz="-0.0880230019550541"
+        izz="0.931256676518883" />
     </inertial>
     <visual>
@@ -466,8 +413,8 @@
     type="continuous">
     <origin
-      xyz="0 0.05 0"
-      rpy="3.14158142866165 1.57079625081358 3.14158142866183" />
-    <parent
-      link="arm_connector_link" />
+      xyz="-0.409742672306299 0.248387046108564 0.660376290839812"
+      rpy="1.57079632680359 0.000114907553872355 1.57079640245869" />
+    <parent
+      link="base_link" />
     <child
       link="arm_base_link" />
@@ -479,15 +426,15 @@
     <inertial>
       <origin
-        xyz="-0.220104658305914 -2.01750447683113E-05 -9.56656233397357E-08"
-        rpy="0 0 0" />
-      <mass
-        value="27.8487184691269" />
-      <inertia
-        ixx="0.139923261741666"
-        ixy="1.06663227751021E-05"
-        ixz="-1.12563617274536E-06"
-        iyy="0.826397782924963"
-        iyz="7.66617430666479E-07"
-        izz="0.851756221048375" />
+        xyz="-0.0372792279944005 0.426695142555641 -0.479484473911662"
+        rpy="0 0 0" />
+      <mass
+        value="45.531535202482" />
+      <inertia
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
Commit message: Fixed issues with passing the wrong joint angles into Jacobian utils. Increased epsilon size to solve singularity issue. Added script for ik validation with circular trajectory

File: aircraft_inspection_robot/urdf/aircraft_inspection_robot.urdf.xacro (robot description, xacro)
@@ -192,4 +192,5 @@
         rpy="0 0 0" />
       <geometry>
+        <!-- <cylinder radius="0.2534" length="0.2032"/> -->
         <mesh
           filename="package://aircraft_inspection_robot/meshes/front_right_wheel_link.STL" />
@@ -208,5 +209,5 @@
       link="front_right_wheel_link" />
     <axis
-      xyz="0 0 0.999999999978938" />
+      xyz="0 0 1" />
   </joint>
   <link
@@ -245,4 +246,5 @@
         rpy="0 0 0" />
       <geometry>
+        <!-- <cylinder radius="0.2534" length="0.2032"/> -->
         <mesh
           filename="package://aircraft_inspection_robot/meshes/front_left_wheel_link.STL" />
@@ -298,4 +300,5 @@
         rpy="0 0 0" />
       <geometry>
+        <!-- <cylinder radius="0.2534" length="0.2032"/> -->
         <mesh
           filename="package://aircraft_inspection_robot/meshes/back_right_wheel_link.STL" />
@@ -351,4 +354,5 @@
         rpy="0 0 0" />
       <geometry>
+        <!-- <cylinder radius="0.2534" length="0.2032"/> -->
         <mesh
           filename="package://aircraft_inspection_robot/meshes/back_left_wheel_link.STL" />
@@ -367,5 +371,5 @@
       link="back_left_wheel_link" />
     <axis
-      xyz="0 0 0.999999999993264" />
+      xyz="0 0 1" />
   </joint>
   <link
@@ -738,5 +742,5 @@
       link="camera_link" />
     <axis
-      xyz="0 0.999999993398127 0.00011490755350285" />
+      xyz="0 1 0" />
   </joint>
   <gazebo>
@@ -801,4 +805,10 @@
         <state_interface name="position"/>
         <state_interface name="velocity"/>
+        <!-- <command_interface name="velocity">
+            <param name="min">-1000.0</param>
+            <param name="max">1000.0</param>
+        </command_interface>
+        <state_interface name="position"/>
+        <state_interface name="velocity"/> -->
     </joint>
     <joint name="arm_link_1_joint">
@@ -809,4 +819,10 @@
         <state_interface name="position"/>
         <state_interface name="velocity"/>
+        <!-- <command_interface name="velocity">
+            <param name="min">-1000.0</param>
+            <param name="max">1000.0</param>
+        </command_interface>
+        <state_interface name="position"/>
+        <state_interface name="velocity"/> -->
     </joint>
     <joint name="arm_link_2_joint">
@@ -817,4 +833,10 @@
         <state_interface name="position"/>
         <state_interface name="velocity"/>
+        <!-- <command_interface name="velocity">
+            <param name="min">-1000.0</param>
+            <param name="max">1000.0</param>
+        </command_interface>
+        <state_interface name="position"/>
+        <state_interface name="velocity"/> -->
     </joint>
     <joint name="arm_link_3_joint">
@@ -825,4 +847,10 @@
         <state_interface name="position"/>
         <state_interface name="velocity"/>
+        <!-- <command_interface name="velocity">
+            <param name="min">-1000.0</param>
+            <param name="max">1000.0</param>
+        </command_interface>
+        <state_interface name="position"/>
+        <state_interface name="velocity"/> -->
     </joint>
     <joint name="arm_link_4_joint">
@@ -833,4 +861,10 @@
         <state_interface name="position"/>
         <state_interface name="velocity"/>
+        <!-- <command_interface name="velocity">
+            <param name="min">-1000.0</param>
+            <param name="max">1000.0</param>
+        </command_interface>
+        <state_interface name="position"/>
+        <state_interface name="velocity"/> -->
     </joint>
     <joint name="arm_link_5_joint">
@@ -841,4 +875,10 @@
         <state_interface name="position"/>
         <state_interface name="velocity"/>
+        <!-- <command_interface name="velocity">
+            <param name="min">-1000.0</param>
+            <param name="max">1000.0</param>
+        </command_interface>
+        <state_interface name="position"/>
+        <state_interface name="velocity"/> -->
     </joint>
   </ros2_control>
@@ -855,5 +895,5 @@
       <pose>0.0 0.0 0.0 0 0 0</pose>
       <always_on>true</always_on>
-      <visualize>true</visualize>
+      <visualize>false</visualize>
       <update_rate>5</update_rate>
       <ray>
@@ -897,5 +937,5 @@
       <pose>0.0 0.0 0.0 0 0 0</pose>
       <always_on>true</always_on>
-      <visualize>true</visualize>
+      <visualize>false</visualize>
       <update_rate>5</update_rate>
       <ray>
@@ -931,5 +971,5 @@
   <link name="depth_camera_sensor_link"></link>
   <joint name="depth_camera_sensor_joint" type="fixed">
-    <origin rpy="-1.571 0 0" xyz="0.2 0 0" />
+    <origin rpy="-1.571 0 0" xyz="1.3 0 0" />
     <parent link="camera_link"/>
     <child link="depth_camera_sensor_link"/>

Commit message: Tried to remove friction on wheel links

File: aircraft_inspection_robot/urdf/aircraft_inspection_robot.urdf.xacro (robot description, xacro)
@@ -757,4 +757,24 @@
       <publish_odom_tf>true</publish_odom_tf>
     </plugin>
+  </gazebo>
+  <gazebo reference="front_right_wheel_link">
+    <material>Gazebo/Black</material>
+    <mu1 value="0.001"/>
+    <mu2 value="0.001"/>
+  </gazebo>
+  <gazebo reference="front_left_wheel_link">
+    <material>Gazebo/Black</material>
+    <mu1 value="0.001"/>
+    <mu2 value="0.001"/>
+  </gazebo>
+  <gazebo reference="back_right_wheel_link">
+    <material>Gazebo/Black</material>
+    <mu1 value="0.001"/>
+    <mu2 value="0.001"/>
+  </gazebo>
+  <gazebo reference="back_left_wheel_link">
+    <material>Gazebo/Black</material>
+    <mu1 value="0.001"/>
+    <mu2 value="0.001"/>
   </gazebo>
   <!-- ROS Gazebo controls -->
