Commit message: Replaced planar movement with skid drive manually implemented

File: aircraft_inspection_robot/urdf/aircraft_inspection_robot.urdf.xacro (robot description, xacro)
@@ -13,5 +13,5 @@
         rpy="0 0 0" />
       <mass
-        value="52.3239752391313" />
+        value="152.3239752391313" />
       <inertia
         ixx="0.952539519630922"
@@ -192,7 +192,7 @@
         rpy="0 0 0" />
       <geometry>
-        <!-- <cylinder radius="0.2534" length="0.2032"/> -->
-        <mesh
-          filename="package://aircraft_inspection_robot/meshes/front_right_wheel_link.STL" />
+        <cylinder radius="0.2281" length="0.2032"/>
+        <!-- <mesh
+          filename="package://aircraft_inspection_robot/meshes/front_right_wheel_link.STL" /> -->
       </geometry>
     </collision>
@@ -215,5 +215,5 @@
     <inertial>
       <origin
-        xyz="1.06668829737838E-07 -1.81805510673927E-07 -0.674003005040707"
+        xyz="1.06668829737838E-07 -1.81805510673927E-07 -0.102621158507274"
         rpy="0 0 0" />
       <mass
@@ -232,6 +232,7 @@
         rpy="0 0 0" />
       <geometry>
-        <mesh
-          filename="package://aircraft_inspection_robot/meshes/front_left_wheel_link.STL" />
+        <cylinder radius="0.2281" length="0.2032"/>
+        <!-- <mesh
+          filename="package://aircraft_inspection_robot/meshes/front_left_wheel_link.STL" /> -->
       </geometry>
       <material
@@ -246,7 +247,7 @@
         rpy="0 0 0" />
       <geometry>
-        <!-- <cylinder radius="0.2534" length="0.2032"/> -->
-        <mesh
-          filename="package://aircraft_inspection_robot/meshes/front_left_wheel_link.STL" />
+        <cylinder radius="0.2281" length="0.2032"/>
+        <!-- <mesh
+          filename="package://aircraft_inspection_robot/meshes/front_left_wheel_link.STL" /> -->
       </geometry>
     </collision>
@@ -256,5 +257,5 @@
     type="continuous">
     <origin
-      xyz="-0.117597527933808 -0.0373680425515616 0.10160911911045"
+      xyz="-0.117597527933808 0.67 0.10160911911045"
       rpy="1.57056878031369 -1.04143176730992 0.000196477434083904" />
     <parent
@@ -300,7 +301,7 @@
         rpy="0 0 0" />
       <geometry>
-        <!-- <cylinder radius="0.2534" length="0.2032"/> -->
-        <mesh
-          filename="package://aircraft_inspection_robot/meshes/back_right_wheel_link.STL" />
+        <cylinder radius="0.2281" length="0.2032"/>
+        <!-- <mesh
+          filename="package://aircraft_inspection_robot/meshes/back_right_wheel_link.STL" /> -->
       </geometry>
     </collision>
@@ -323,5 +324,5 @@
     <inertial>
       <origin
-        xyz="1.29034836829356E-07 -2.66555836092586E-06 -0.673983123389094"
+        xyz="1.29034836829356E-07 -2.66555836092586E-06 -0.102621158507274"
         rpy="0 0 0" />
       <mass
@@ -340,6 +341,7 @@
         rpy="0 0 0" />
       <geometry>
-        <mesh
-          filename="package://aircraft_inspection_robot/meshes/back_left_wheel_link.STL" />
+        <cylinder radius="0.2281" length="0.2032"/>
+        <!-- <mesh
+          filename="package://aircraft_inspection_robot/meshes/back_left_wheel_link.STL" /> -->
       </geometry>
       <material
@@ -354,7 +356,7 @@
         rpy="0 0 0" />
       <geometry>
-        <!-- <cylinder radius="0.2534" length="0.2032"/> -->
-        <mesh
-          filename="package://aircraft_inspection_robot/meshes/back_left_wheel_link.STL" />
+        <cylinder radius="0.2281" length="0.2032"/>
+        <!-- <mesh
+          filename="package://aircraft_inspection_robot/meshes/back_left_wheel_link.STL" /> -->
       </geometry>
     </collision>
@@ -364,5 +366,5 @@
     type="continuous">
     <origin
-      xyz="-0.701797527935311 -0.0373482051170577 0.101609112969085"
+      xyz="-0.701797527935311 0.67 0.101609112969085"
       rpy="1.56727528936655 -1.5381898923507 0.00352290998991109" />
     <parent
@@ -744,5 +746,5 @@
       xyz="0 1 0" />
   </joint>
-  <gazebo>
+  <!-- <gazebo>
     <plugin name="object_controller" filename="libgazebo_ros_planar_move.so">
       <ros>
@@ -757,6 +759,6 @@
       <publish_odom_tf>true</publish_odom_tf>
     </plugin>
-  </gazebo>
-  <gazebo reference="front_right_wheel_link">
+  </gazebo> -->
+  <!-- <gazebo reference="front_right_wheel_link">
     <material>Gazebo/Black</material>
     <mu1 value="0.001"/>
@@ -777,5 +779,5 @@
     <mu1 value="0.001"/>
     <mu2 value="0.001"/>
-  </gazebo>
+  </gazebo> -->
   <!-- ROS Gazebo controls -->
   <ros2_control name="GazeboSystem" type="system">
@@ -785,5 +787,5 @@
     <!-- Velocity controllers -->
     <!-- Front Wheels -->
-    <!-- <joint name="front_right_wheel_joint">
+    <joint name="front_right_wheel_joint">
         <command_interface name="velocity">
             <param name="min">-1000.0</param>
@@ -816,5 +818,5 @@
         <state_interface name="position"/>
         <state_interface name="velocity"/>
-    </joint> -->
+    </joint>
     <!-- Position Controllers -->
     <joint name="arm_base_joint">
