Commit message: Added custom aircraft and apriltag world

File: aircraft_inspection_robot/urdf/aircraft_inspection_robot.urdf copy.xacro (robot description, xacro)
@@ -906,4 +906,122 @@
     </joint>
   </ros2_control>
+  <!-- Sensors -->
+  <!-- Front LiDAR -->
+  <link name="front_lidar_sensor_link"></link>
+  <joint name="front_lidar_sensor_joint" type="fixed">
+    <origin rpy="1.571 1.571 0" xyz="0 -0.05 0" />
+    <parent link="front_lidar_link"/>
+    <child link="front_lidar_sensor_link"/>
+  </joint>
+  <gazebo reference="front_lidar_sensor_link">
+    <sensor name="front_lidar" type="ray">
+      <pose>0.0 0.0 0.0 0 0 0</pose>
+      <always_on>true</always_on>
+      <visualize>true</visualize>
+      <update_rate>5</update_rate>
+      <ray>
+        <scan>
+          <horizontal>
+            <samples>360</samples>
+            <resolution>1.00000</resolution>
+            <min_angle>-0.5</min_angle>
+            <max_angle>3.54</max_angle>
+          </horizontal>
+        </scan>
+        <range>
+          <min>0.16</min>
+          <max>10.0</max>
+          <resolution>0.015000</resolution>
+        </range>
+        <noise>
+          <type>gaussian</type>
+          <mean>0.0</mean>
+          <stddev>0.01</stddev>
+        </noise>
+      </ray>
+      <plugin name="front_scan" filename="libgazebo_ros_ray_sensor.so">
+        <ros>
+          <remapping>~/out:=front_scan</remapping>
+        </ros>
+        <output_type>sensor_msgs/LaserScan</output_type>
+        <frame_name>front_lidar_sensor_link</frame_name>
+      </plugin>
+    </sensor>
+  </gazebo>
+  <!-- Rear LiDAR -->
+  <link name="rear_lidar_sensor_link"></link>
+  <joint name="rear_lidar_sensor_joint" type="fixed">
+    <origin rpy="1.571 1.571 0" xyz="0 -0.05 0" />
+    <parent link="rear_lidar_link"/>
+    <child link="rear_lidar_sensor_link"/>
+  </joint>
+  <gazebo reference="rear_lidar_sensor_link">
+    <sensor name="rear_lidar" type="ray">
+      <pose>0.0 0.0 0.0 0 0 0</pose>
+      <always_on>true</always_on>
+      <visualize>true</visualize>
+      <update_rate>5</update_rate>
+      <ray>
+        <scan>
+          <horizontal>
+            <samples>360</samples>
+            <resolution>1.00000</resolution>
+            <min_angle>-0.5</min_angle>
+            <max_angle>3.54</max_angle>
+          </horizontal>
+        </scan>
+        <range>
+          <min>0.16</min>
+          <max>10.0</max>
+          <resolution>0.015000</resolution>
+        </range>
+        <noise>
+          <type>gaussian</type>
+          <mean>0.0</mean>
+          <stddev>0.01</stddev>
+        </noise>
+      </ray>
+      <plugin name="rear_scan" filename="libgazebo_ros_ray_sensor.so">
+        <ros>
+          <remapping>~/out:=rear_scan</remapping>
+        </ros>
+        <output_type>sensor_msgs/LaserScan</output_type>
+        <frame_name>rear_lidar_sensor_link</frame_name>
+      </plugin>
+    </sensor>
+  </gazebo>
+  <!-- Depth Camera -->
+  <link name="depth_camera_sensor_link"></link>
+  <joint name="depth_camera_sensor_joint" type="fixed">
+    <origin rpy="-1.571 0 0" xyz="0.2 0 0" />
+    <parent link="camera_link"/>
+    <child link="depth_camera_sensor_link"/>
+  </joint>
+  <gazebo reference="depth_camera_sensor_link">
+    <sensor name="depth_camera" type="depth">
+      <camera name="depth_camera">
+        <!-- Camera properties -->
+        <horizontal_fov>1.047</horizontal_fov>
+        <vertical_fov>0.785</vertical_fov>
+        <image>
+          <width>640</width>
+          <height>480</height>
+        </image>
+        <clip>
+          <near>0.1</near>
+          <far>20.0</far>
+        </clip>
+      </camera>
+      <!-- Depth camera Gazebo plugin -->
+      <plugin name="gazebo_ros_depth_camera" filename="libgazebo_ros_camera.so">
+        <alwaysOn>true</alwaysOn>
+        <updateRate>30.0</updateRate>
+        <cameraName>depth</cameraName>
+        <frameName>depth_camera_sensor_link</frameName>
+        <imageTopicName>image_raw</imageTopicName>
+        <cameraInfoTopicName>camera_info</cameraInfoTopicName>
+      </plugin>
+    </sensor>
+  </gazebo>
   <gazebo>
     <plugin filename="libgazebo_ros2_control.so" name="gazebo_ros2_control">

File: aircraft_inspection_robot/urdf/aircraft_inspection_robot.urdf.xacro (robot description, xacro)
@@ -10,15 +10,15 @@
     <inertial>
       <origin
-        xyz="-0.409821173833434 0.248346984053139 0.186905789650059"
-        rpy="0 0 0" />
-      <mass
-        value="16.3100062980245" />
-      <inertia
-        ixx="0.442677686543008"
-        ixy="-4.25661758844677E-05"
-        ixz="-8.01477308223399E-09"
-        iyy="1.88352843223116"
-        iyz="1.6365434477415E-05"
-        izz="2.08653679036228" />
+        xyz="-0.409737523113878 0.248339713620131 0.209639401630241"
+        rpy="0 0 0" />
+      <mass
+        value="52.4458402259021" />
+      <inertia
+        ixx="1.61796946709653"
+        ixy="-4.26019586297761E-05"
+        ixz="5.36565329733604E-05"
+        iyy="3.60901877519089"
+        iyz="0.00014045219036093"
+        izz="4.89191044456781" />
     </inertial>
     <visual>
@@ -52,4 +52,110 @@
   </joint>
   <link
+    name="front_lidar_link">
+    <inertial>
+      <origin
+        xyz="-0.00725498730999624 -0.159524096445023 -5.18934305249186E-08"
+        rpy="0 0 0" />
+      <mass
+        value="21.0173459101461" />
+      <inertia
+        ixx="0.360630213819554"
+        ixy="-0.0108096413980878"
+        ixz="4.79803425565932E-08"
+        iyy="0.186912416456727"
+        iyz="-2.37737605206146E-07"
+        izz="0.361463047566562" />
+    </inertial>
+    <visual>
+      <origin
+        xyz="0 0 0"
+        rpy="0 0 0" />
+      <geometry>
+        <mesh
+          filename="package://aircraft_inspection_robot/meshes/front_lidar_link.STL" />
+      </geometry>
+      <material
+        name="">
+        <color
+          rgba="0.792156862745098 0.819607843137255 0.933333333333333 1" />
+      </material>
+    </visual>
+    <collision>
+      <origin
+        xyz="0 0 0"
+        rpy="0 0 0" />
+      <geometry>
+        <mesh
+          filename="package://aircraft_inspection_robot/meshes/front_lidar_link.STL" />
+      </geometry>
+    </collision>
+  </link>
+  <joint
+    name="front_lidar_joint"
+    type="fixed">
+    <origin
+      xyz="0.308106449560569 0.248338347564378 0.236097315694741"
+      rpy="-1.57091123434865 0 0" />
+    <parent
+      link="base_link" />
+    <child
+      link="front_lidar_link" />
+    <axis
+      xyz="0 0 0" />
+  </joint>
+  <link
+    name="rear_lidar_link">
+    <inertial>
+      <origin
+        xyz="-0.00725498516150735 0.1695240965549 -5.18932890547497E-08"
+        rpy="0 0 0" />
+      <mass
+        value="21.0173459127111" />
+      <inertia
+        ixx="0.360630214140233"
+        ixy="-0.0108096390967668"
+        ixz="4.79968519505956E-08"
+        iyy="0.18691241620145"
+        iyz="-2.37742872890824E-07"
+        izz="0.361463047569039" />
+    </inertial>
+    <visual>
+      <origin
+        xyz="0 0 0"
+        rpy="0 0 0" />
+      <geometry>
+        <mesh
+          filename="package://aircraft_inspection_robot/meshes/rear_lidar_link.STL" />
+      </geometry>
+      <material
+        name="">
+        <color
+          rgba="0.792156862745098 0.819607843137255 0.933333333333333 1" />
+      </material>
+    </visual>
+    <collision>
+      <origin
+        xyz="0 0 0"
+        rpy="0 0 0" />
+      <geometry>
+        <mesh
+          filename="package://aircraft_inspection_robot/meshes/rear_lidar_link.STL" />
+      </geometry>
+    </collision>
+  </link>
+  <joint
+    name="rear_lidar_joint"
+    type="fixed">
+    <origin
+      xyz="0.308106449560569 0.248338347564378 0.236097315694741"
+      rpy="-1.57068141924114 0 3.14159265358979" />
+    <parent
+      link="base_link" />
+    <child
+      link="rear_lidar_link" />
+    <axis
+      xyz="0 0 0" />
+  </joint>
+  <link
     name="front_right_wheel_link">
     <inertial>
@@ -61,8 +167,8 @@
       <inertia
         ixx="0.267032855143768"
-        ixy="-1.12646160247748E-12"
-        ixz="-5.64889033632766E-10"
+        ixy="-1.12643384679206E-12"
+        ixz="-5.64889032158929E-10"
         iyy="0.267032853623031"
-        iyz="9.3846814728935E-12"
+        iyz="9.3846801464399E-12"
         izz="0.388719266107455" />
     </inertial>
@@ -90,13 +196,4 @@
       </geometry>
     </collision>
-    <friction>
-      <ode>
-        <mu>0.0</mu> <!-- Friction coefficient -->
-        <mu2>0.0</mu2> <!-- Second friction coefficient (optional) -->
-        <fdir1>0 0 0</fdir1> <!-- Friction direction (optional) -->
-        <slip1>0.0</slip1> <!-- Slip coefficient for friction direction 1 (optional) -->
-        <slip2>0.0</slip2> <!-- Slip coefficient for friction direction 2 (optional) -->
-      </ode>
-    </friction>
   </link>
   <joint
@@ -117,5 +214,5 @@
     <inertial>
       <origin
-        xyz="-6.09432209558447E-14 1.71113179181503E-10 -0.10313316315041"
+        xyz="-6.06656651996884E-14 1.71113873070894E-10 -0.10313316315041"
         rpy="0 0 0" />
       <mass
@@ -123,8 +220,8 @@
       <inertia
         ixx="0.267032855143761"
-        ixy="-1.14495324380602E-12"
-        ixz="5.64901636627518E-10"
+        ixy="-1.14495324383746E-12"
+        ixz="5.64901635417955E-10"
         iyy="0.267032853623031"
-        iyz="-9.3691461263112E-12"
+        iyz="-9.36914437972927E-12"
         izz="0.388719266107462" />
     </inertial>
@@ -152,13 +249,4 @@
       </geometry>
     </collision>
-    <friction>
-      <ode>
-        <mu>0.0</mu> <!-- Friction coefficient -->
-        <mu2>0.0</mu2> <!-- Second friction coefficient (optional) -->
-        <fdir1>0 0 0</fdir1> <!-- Friction direction (optional) -->
-        <slip1>0.0</slip1> <!-- Slip coefficient for friction direction 1 (optional) -->
-        <slip2>0.0</slip2> <!-- Slip coefficient for friction direction 2 (optional) -->
-      </ode>
-    </friction>
   </link>
   <joint
@@ -166,5 +254,5 @@
     type="continuous">
     <origin
-      xyz="-0.117597571165592 0.533998775516627 0.101543464746799"
+      xyz="-0.117597571165592 0.533998775516627 0.101543464746798"
       rpy="1.57061905476483 -0.865579426080518 0.00013506316993608" />
     <parent
@@ -179,14 +267,14 @@
     <inertial>
       <origin
-        xyz="-6.0507154842071E-14 1.71112790603445E-10 0.103133072201983"
-        rpy="0 0 0" />
-      <mass
-        value="17.0942965183762" />
+        xyz="-6.03961325396085E-14 1.71112679581142E-10 0.103133072201983"
+        rpy="0 0 0" />
+      <mass
+        value="17.0942965183763" />
       <inertia
         ixx="0.267032855143761"
-        ixy="-1.14615484329692E-12"
-        ixz="-5.64900111493875E-10"
+        ixy="-1.14615484325525E-12"
+        ixz="-5.64900110911116E-10"
         iyy="0.267032853623031"
-        iyz="9.36830934754481E-12"
+        iyz="9.36830792283539E-12"
         izz="0.388719266107461" />
     </inertial>
@@ -214,13 +302,4 @@
       </geometry>
     </collision>
-    <friction>
-      <ode>
-        <mu>0.0</mu> <!-- Friction coefficient -->
-        <mu2>0.0</mu2> <!-- Second friction coefficient (optional) -->
-        <fdir1>0 0 0</fdir1> <!-- Friction direction (optional) -->
-        <slip1>0.0</slip1> <!-- Slip coefficient for friction direction 1 (optional) -->
-        <slip2>0.0</slip2> <!-- Slip coefficient for friction direction 2 (optional) -->
-      </ode>
-    </friction>
   </link>
   <joint
@@ -228,6 +307,6 @@
     type="continuous">
     <origin
-      xyz="-0.701797527934933 -0.0373531949241711 0.101609113542451"
-      rpy="1.57061607230749 -0.879581000000789 0.000138956671881705" />
+      xyz="-0.7018 -0.037353 0.10161"
+      rpy="1.5706 -0.87958 0.00013896" />
     <parent
       link="base_link" />
@@ -241,5 +320,5 @@
     <inertial>
       <origin
-        xyz="-5.73430192218893E-14 1.71111458335815E-10 -0.103131061396203"
+        xyz="-5.65658631046517E-14 1.71111347313513E-10 -0.103131061396203"
         rpy="0 0 0" />
       <mass
@@ -247,8 +326,8 @@
       <inertia
         ixx="0.267032855143766"
-        ixy="-1.12798336651991E-12"
-        ixz="5.64892005341136E-10"
+        ixy="-1.12798336645332E-12"
+        ixz="5.64892007313028E-10"
         iyy="0.267032853623031"
-        iyz="-9.37929450597929E-12"
+        iyz="-9.37929468555027E-12"
         izz="0.388719266107457" />
     </inertial>
@@ -276,13 +355,4 @@
       </geometry>
     </collision>
-    <friction>
-      <ode>
-        <mu>0.0</mu> <!-- Friction coefficient -->
-        <mu2>0.0</mu2> <!-- Second friction coefficient (optional) -->
-        <fdir1>0 0 0</fdir1> <!-- Friction direction (optional) -->
-        <slip1>0.0</slip1> <!-- Slip coefficient for friction direction 1 (optional) -->
-        <slip2>0.0</slip2> <!-- Slip coefficient for friction direction 2 (optional) -->
-      </ode>
-    </friction>
   </link>
   <joint
@@ -290,6 +360,6 @@
     type="continuous">
     <origin
-      xyz="-0.70179757116575 0.534000833067587 0.101543460648476"
-      rpy="-1.57057031157129 -1.03746333162058 3.14139810362434" />
+      xyz="-0.7018 0.534 0.10154"
+      rpy="-1.5706 -1.0375 3.1414" />
     <parent
       link="base_link" />
@@ -300,26 +370,26 @@
   </joint>
   <link
-    name="top_plate_link">
-    <inertial>
-      <origin
-        xyz="-2.90134583025292E-11 0.00438783814695193 3.83026943495679E-15"
-        rpy="0 0 0" />
-      <mass
-        value="16.7771592854839" />
-      <inertia
-        ixx="1.09903225464032"
-        ixy="-1.03404210583146E-08"
-        ixz="3.53674468306753E-08"
-        iyy="2.66325912479572"
-        iyz="1.7337070364401E-15"
-        izz="1.566461199065" />
-    </inertial>
-    <visual>
-      <origin
-        xyz="0 0 0"
-        rpy="0 0 0" />
-      <geometry>
-        <mesh
-          filename="package://aircraft_inspection_robot/meshes/top_plate_link.STL" />
+    name="arm_connector_link">
+    <inertial>
+      <origin
+        xyz="-1.43143330522122E-10 0.0216537321612436 1.10744746706359E-14"
+        rpy="0 0 0" />
+      <mass
+        value="2.62877306618386" />
+      <inertia
+        ixx="0.0207836884851897"
+        ixy="-1.25135931667707E-10"
+        ixz="-2.20944162334301E-25"
+        iyy="0.039713380262994"
+        iyz="-2.37404276874067E-17"
+        izz="0.0207836884851897" />
+    </inertial>
+    <visual>
+      <origin
+        xyz="0 0 0"
+        rpy="0 0 0" />
+      <geometry>
+        <mesh
+          filename="package://aircraft_inspection_robot/meshes/arm_connector_link.STL" />
       </geometry>
       <material
@@ -335,18 +405,18 @@
       <geometry>
         <mesh
-          filename="package://aircraft_inspection_robot/meshes/top_plate_link.STL" />
-      </geometry>
-    </collision>
-  </link>
-  <joint
-    name="top_plate_joint"
+          filename="package://aircraft_inspection_robot/meshes/arm_connector_link.STL" />
+      </geometry>
+    </collision>
+  </link>
+  <joint
+    name="arm_connect_joint"
     type="fixed">
     <origin
-      xyz="-0.409697551607141 0.248358589255724 0.412726287085218"
-      rpy="1.57068141924114 0 0" />
+      xyz="-0.4097 0.24836 0.41908"
+      rpy="1.5707 0 0" />
     <parent
       link="base_link" />
     <child
-      link="top_plate_link" />
+      link="arm_connector_link" />
     <axis
       xyz="0 0 0" />
@@ -356,5 +426,5 @@
     <inertial>
       <origin
-        xyz="1.39083189409916E-13 0.164974567451517 -1.15671067169032E-09"
+        xyz="8.98447982677908E-14 0.118624566442621 -7.84175280266197E-10"
         rpy="0 0 0" />
       <mass
@@ -362,8 +432,8 @@
       <inertia
         ixx="0.278054099642839"
-        ixy="-4.4034337604742E-14"
-        ixz="1.17918737185581E-16"
+        ixy="-4.40146949106952E-14"
+        ixz="1.13856898220502E-16"
         iyy="0.226366310502593"
-        iyz="6.24174992555768E-10"
+        iyz="6.241749681372E-10"
         izz="0.320787148766728" />
     </inertial>
@@ -396,8 +466,8 @@
     type="continuous">
     <origin
-      xyz="0 0.01 0"
-      rpy="3.14158139197888 1.57079625081358 3.14158139197905" />
-    <parent
-      link="top_plate_link" />
+      xyz="0 0.05 0"
+      rpy="3.14158142866165 1.57079625081358 3.14158142866183" />
+    <parent
+      link="arm_connector_link" />
     <child
       link="arm_base_link" />
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