Commit message: Updated mass values to try to fix joint explosion issue but didn't fully solve it

File: aircraft_inspection_robot/urdf/aircraft_inspection_robot.urdf copy.xacro (robot description, xacro)
@@ -10,15 +10,15 @@
     <inertial>
       <origin
-        xyz="-0.409737523113878 0.248339713620131 0.209639401630241"
-        rpy="0 0 0" />
-      <mass
-        value="52.4458402259021" />
-      <inertia
-        ixx="1.61796946709653"
-        ixy="-4.26019586297761E-05"
-        ixz="5.36565329733604E-05"
-        iyy="3.60901877519089"
-        iyz="0.00014045219036093"
-        izz="4.89191044456781" />
+        xyz="-0.40974645535857 0.24834344494391 0.242010590101945"
+        rpy="0 0 0" />
+      <mass
+        value="352.3239752391313" />
+      <inertia
+        ixx="0.952539519630922"
+        ixy="-4.26200364814785E-05"
+        ixz="5.36575380324012E-05"
+        iyy="30.80199276879049"
+        iyz="2.4370448304257E-05"
+        izz="40.07464899613958" />
     </inertial>
     <visual>
@@ -33,5 +33,5 @@
         name="">
         <color
-          rgba="1 1 1 1" />
+          rgba="0.250980392156863 0.250980392156863 0.250980392156863 1" />
       </material>
     </visual>
@@ -55,15 +55,15 @@
     <inertial>
       <origin
-        xyz="-0.00725498730999624 -0.159524096445023 -5.18934305249186E-08"
-        rpy="0 0 0" />
-      <mass
-        value="21.0173459101461" />
-      <inertia
-        ixx="0.360630213819554"
-        ixy="-0.0108096413980878"
-        ixz="4.79803425565932E-08"
-        iyy="0.186912416456727"
-        iyz="-2.37737605206146E-07"
-        izz="0.361463047566562" />
+        xyz="-0.00725496120108809 -0.159524101399661 -5.98196165102483E-08"
+        rpy="0 0 0" />
+      <mass
+        value="2.62716823876827" />
+      <inertia
+        ixx="0.0112696941818608"
+        ixy="-0.00033780129369249"
+        ixz="1.4993857049244E-09"
+        iyy="0.00584101301427301"
+        iyz="-7.42930015937879E-09"
+        izz="0.0112957202364551" />
     </inertial>
     <visual>
@@ -95,5 +95,5 @@
     type="fixed">
     <origin
-      xyz="0.308106449560569 0.248338347564378 0.236097315694741"
+      xyz="0.252189298222892 0.248326110601867 0.129347762825463"
       rpy="-1.57091123434865 0 0" />
     <parent
@@ -108,15 +108,15 @@
     <inertial>
       <origin
-        xyz="-0.00725498516150735 0.1695240965549 -5.18932890547497E-08"
-        rpy="0 0 0" />
-      <mass
-        value="21.0173459127111" />
-      <inertia
-        ixx="0.360630214140233"
-        ixy="-0.0108096390967668"
-        ixz="4.79968519505956E-08"
-        iyy="0.18691241620145"
-        iyz="-2.37742872890824E-07"
-        izz="0.361463047569039" />
+        xyz="-0.00725495907227769 -0.159524101502578 -5.98195511736233E-08"
+        rpy="0 0 0" />
+      <mass
+        value="2.62716823908889" />
+      <inertia
+        ixx="0.0112696941918823"
+        ixy="-0.000337801221774006"
+        ixz="1.49990162575632E-09"
+        iyy="0.00584101300629532"
+        iyz="-7.42946478333022E-09"
+        izz="0.0112957202365325" />
     </inertial>
     <visual>
@@ -148,5 +148,5 @@
     type="fixed">
     <origin
-      xyz="0.308106449560569 0.248338347564378 0.236097315694741"
+      xyz="-1.07167463581468 0.248325943235427 0.129347754093208"
       rpy="-1.57068141924114 0 3.14159265358979" />
     <parent
@@ -161,15 +161,15 @@
     <inertial>
       <origin
-        xyz="-5.59829960167235E-14 1.71109293400917E-10 0.103131389958602"
-        rpy="0 0 0" />
-      <mass
-        value="17.0942965183764" />
-      <inertia
-        ixx="0.267032855143768"
-        ixy="-1.12643384679206E-12"
-        ixz="-5.64889032158929E-10"
-        iyy="0.267032853623031"
-        iyz="9.3846801464399E-12"
-        izz="0.388719266107455" />
+        xyz="7.69611511519663E-07 -1.70468712881733E-07 0.102621158507274"
+        rpy="0 0 0" />
+      <mass
+        value="26.0461976105726" />
+      <inertia
+        ixx="0.285954065616882"
+        ixy="7.95282541629767E-07"
+        ixz="1.27020782265502E-07"
+        iyy="0.28595474175216"
+        iyz="-3.78487432157488E-07"
+        izz="0.40415282922357" />
     </inertial>
     <visual>
@@ -184,14 +184,15 @@
         name="">
         <color
-          rgba="0.250980392156863 0.250980392156863 0.250980392156863 1" />
-      </material>
-    </visual>
-    <collision>
-      <origin
-        xyz="0 0 0"
-        rpy="0 0 0" />
-      <geometry>
-        <mesh
-          filename="package://aircraft_inspection_robot/meshes/front_right_wheel_link.STL" />
+          rgba="0.792156862745098 0.819607843137255 0.933333333333333 1" />
+      </material>
+    </visual>
+    <collision>
+      <origin
+        xyz="0 0 0"
+        rpy="0 0 0" />
+      <geometry>
+        <cylinder radius="0.2281" length="0.2032"/>
+        <!-- <mesh
+          filename="package://aircraft_inspection_robot/meshes/front_right_wheel_link.STL" /> -->
       </geometry>
     </collision>
@@ -201,6 +202,6 @@
     type="continuous">
     <origin
-      xyz="-0.117597527934808 -0.0373548329643068 0.101609117592568"
-      rpy="-1.57057710899586 -1.01905526588804 3.14140604048142" />
+      xyz="-0.117597527933808 -0.0373680425515616 0.10160911911045"
+      rpy="-1.57068160265985 -0.0571716575997457 3.14159265358979" />
     <parent
       link="base_link" />
@@ -214,37 +215,39 @@
     <inertial>
       <origin
-        xyz="-6.06656651996884E-14 1.71113873070894E-10 -0.10313316315041"
-        rpy="0 0 0" />
-      <mass
-        value="17.0942965183763" />
-      <inertia
-        ixx="0.267032855143761"
-        ixy="-1.14495324383746E-12"
-        ixz="5.64901635417955E-10"
-        iyy="0.267032853623031"
-        iyz="-9.36914437972927E-12"
-        izz="0.388719266107462" />
-    </inertial>
-    <visual>
-      <origin
-        xyz="0 0 0"
-        rpy="0 0 0" />
-      <geometry>
-        <mesh
-          filename="package://aircraft_inspection_robot/meshes/front_left_wheel_link.STL" />
-      </geometry>
-      <material
-        name="">
-        <color
-          rgba="0.250980392156863 0.250980392156863 0.250980392156863 1" />
-      </material>
-    </visual>
-    <collision>
-      <origin
-        xyz="0 0 0"
-        rpy="0 0 0" />
-      <geometry>
-        <mesh
-          filename="package://aircraft_inspection_robot/meshes/front_left_wheel_link.STL" />
+        xyz="1.06668829737838E-07 -1.81805510673927E-07 -0.102621158507274"
+        rpy="0 0 0" />
+      <mass
+        value="26.0463242126014" />
+      <inertia
+        ixx="0.285954618303477"
+        ixy="7.68759858498613E-07"
+        ixz="6.28786224972317E-07"
+        iyy="0.285955290913927"
+        iyz="3.7011482934088E-07"
+        izz="0.404153186322765" />
+    </inertial>
+    <visual>
+      <origin
+        xyz="0 0 0"
+        rpy="0 0 0" />
+      <geometry>
+        <cylinder radius="0.2281" length="0.2032"/>
+        <!-- <mesh
+          filename="package://aircraft_inspection_robot/meshes/front_left_wheel_link.STL" /> -->
+      </geometry>
+      <material
+        name="">
+        <color
+          rgba="0.792156862745098 0.819607843137255 0.933333333333333 1" />
+      </material>
+    </visual>
+    <collision>
+      <origin
+        xyz="0 0 0"
+        rpy="0 0 0" />
+      <geometry>
+        <cylinder radius="0.2281" length="0.2032"/>
+        <!-- <mesh
+          filename="package://aircraft_inspection_robot/meshes/front_left_wheel_link.STL" /> -->
       </geometry>
     </collision>
@@ -254,6 +257,6 @@
     type="continuous">
     <origin
-      xyz="-0.117597571165592 0.533998775516627 0.101543464746798"
-      rpy="1.57061905476483 -0.865579426080518 0.00013506316993608" />
+      xyz="-0.117597527933808 0.63 0.10160911911045"
+      rpy="1.57056878031369 -1.04143176730992 0.000196477434083904" />
     <parent
       link="base_link" />
@@ -267,15 +270,15 @@
     <inertial>
       <origin
-        xyz="-6.03961325396085E-14 1.71112679581142E-10 0.103133072201983"
-        rpy="0 0 0" />
-      <mass
-        value="17.0942965183763" />
-      <inertia
-        ixx="0.267032855143761"
-        ixy="-1.14615484325525E-12"
-        ixz="-5.64900110911116E-10"
-        iyy="0.267032853623031"
-        iyz="9.36830792283539E-12"
-        izz="0.388719266107461" />
+        xyz="8.41577684762562E-08 -1.68242609732694E-07 0.102641039115083"
+        rpy="0 0 0" />
+      <mass
+        value="26.0462008072991" />
+      <inertia
+        ixx="0.285954040177974"
+        ixy="7.90067012358279E-07"
+        ixz="-6.50671063736261E-07"
+        iyy="0.285954742544619"
+        iyz="-3.69738156013685E-07"
+        izz="0.40415280236699" />
     </inertial>
     <visual>
@@ -290,14 +293,15 @@
         name="">
         <color
-          rgba="0.250980392156863 0.250980392156863 0.250980392156863 1" />
-      </material>
-    </visual>
-    <collision>
-      <origin
-        xyz="0 0 0"
-        rpy="0 0 0" />
-      <geometry>
-        <mesh
-          filename="package://aircraft_inspection_robot/meshes/back_right_wheel_link.STL" />
+          rgba="0.792156862745098 0.819607843137255 0.933333333333333 1" />
+      </material>
+    </visual>
+    <collision>
+      <origin
+        xyz="0 0 0"
+        rpy="0 0 0" />
+      <geometry>
+        <cylinder radius="0.2281" length="0.2032"/>
+        <!-- <mesh
+          filename="package://aircraft_inspection_robot/meshes/back_right_wheel_link.STL" /> -->
       </geometry>
     </collision>
@@ -307,6 +311,6 @@
     type="continuous">
     <origin
-      xyz="-0.7018 -0.037353 0.10161"
-      rpy="1.5706 -0.87958 0.00013896" />
+      xyz="-0.701797527935311 -0.0373482051170577 0.101609112969085"
+      rpy="1.57064724689163 -0.690734458596981 9.50549862212618E-05" />
     <parent
       link="base_link" />
@@ -320,37 +324,39 @@
     <inertial>
       <origin
-        xyz="-5.65658631046517E-14 1.71111347313513E-10 -0.103131061396203"
-        rpy="0 0 0" />
-      <mass
-        value="17.0942965183761" />
-      <inertia
-        ixx="0.267032855143766"
-        ixy="-1.12798336645332E-12"
-        ixz="5.64892007313028E-10"
-        iyy="0.267032853623031"
-        iyz="-9.37929468555027E-12"
-        izz="0.388719266107457" />
-    </inertial>
-    <visual>
-      <origin
-        xyz="0 0 0"
-        rpy="0 0 0" />
-      <geometry>
-        <mesh
-          filename="package://aircraft_inspection_robot/meshes/back_left_wheel_link.STL" />
-      </geometry>
-      <material
-        name="">
-        <color
-          rgba="0.250980392156863 0.250980392156863 0.250980392156863 1" />
-      </material>
-    </visual>
-    <collision>
-      <origin
-        xyz="0 0 0"
-        rpy="0 0 0" />
-      <geometry>
-        <mesh
-          filename="package://aircraft_inspection_robot/meshes/back_left_wheel_link.STL" />
+        xyz="1.29034836829356E-07 -2.66555836092586E-06 -0.102621158507274"
+        rpy="0 0 0" />
+      <mass
+        value="26.0463122941313" />
+      <inertia
+        ixx="0.285954575528675"
+        ixy="7.71478869336928E-07"
+        ixz="6.45837128179966E-07"
+        iyy="0.285955250948586"
+        iyz="7.90647100387111E-07"
+        izz="0.404153156835058" />
+    </inertial>
+    <visual>
+      <origin
+        xyz="0 0 0"
+        rpy="0 0 0" />
+      <geometry>
+        <cylinder radius="0.2281" length="0.2032"/>
+        <!-- <mesh
+          filename="package://aircraft_inspection_robot/meshes/back_left_wheel_link.STL" /> -->
+      </geometry>
+      <material
+        name="">
+        <color
+          rgba="0.792156862745098 0.819607843137255 0.933333333333333 1" />
+      </material>
+    </visual>
+    <collision>
+      <origin
+        xyz="0 0 0"
+        rpy="0 0 0" />
+      <geometry>
+        <cylinder radius="0.2281" length="0.2032"/>
+        <!-- <mesh
+          filename="package://aircraft_inspection_robot/meshes/back_left_wheel_link.STL" /> -->
       </geometry>
     </collision>
@@ -360,6 +366,6 @@
     type="continuous">
     <origin
-      xyz="-0.7018 0.534 0.10154"
-      rpy="-1.5706 -1.0375 3.1414" />
+      xyz="-0.701797527935311 0.63 0.101609112969085"
+      rpy="1.56727528936655 -1.5381898923507 0.00352290998991109" />
     <parent
       link="base_link" />
@@ -370,71 +376,18 @@
   </joint>
   <link
-    name="arm_connector_link">
-    <inertial>
-      <origin
-        xyz="-1.43143330522122E-10 0.0216537321612436 1.10744746706359E-14"
-        rpy="0 0 0" />
-      <mass
-        value="2.62877306618386" />
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
File: aircraft_inspection_robot/urdf/aircraft_inspection_robot.urdf.xacro (robot description, xacro)
@@ -13,12 +13,12 @@
         rpy="0 0 0" />
       <mass
-        value="152.3239752391313" />
+        value="3520.3239752391313" />
       <inertia
         ixx="0.952539519630922"
         ixy="-4.26200364814785E-05"
         ixz="5.36575380324012E-05"
-        iyy="3.80199276879049"
+        iyy="30.80199276879049"
         iyz="2.4370448304257E-05"
-        izz="4.07464899613958" />
+        izz="40.07464899613958" />
     </inertial>
     <visual>
@@ -257,5 +257,5 @@
     type="continuous">
     <origin
-      xyz="-0.117597527933808 0.67 0.10160911911045"
+      xyz="-0.117597527933808 0.63 0.10160911911045"
       rpy="1.57056878031369 -1.04143176730992 0.000196477434083904" />
     <parent
@@ -366,5 +366,5 @@
     type="continuous">
     <origin
-      xyz="-0.701797527935311 0.67 0.101609112969085"
+      xyz="-0.701797527935311 0.63 0.101609112969085"
       rpy="1.56727528936655 -1.5381898923507 0.00352290998991109" />
     <parent
@@ -427,4 +427,9 @@
     <axis
       xyz="0 1 0" />
+    <pid>
+      <p>1.0</p>
+      <i>0.1</i>
+      <d>0.01</d>
+    </pid>
   </joint>
   <link
@@ -435,5 +440,5 @@
         rpy="0 0 0" />
       <mass
-        value="0.45531535202482" />
+        value="4.5531535202482" />
       <inertia
         ixx="5.83147761609791"
@@ -480,4 +485,9 @@
     <axis
       xyz="0 0 -1" />
+    <pid>
+      <p>1.0</p>
+      <i>0.1</i>
+      <d>0.01</d>
+    </pid>
   </joint>
   <link
@@ -488,5 +498,5 @@
         rpy="0 0 0" />
       <mass
-        value="0.455315352024768" />
+        value="4.55315352024768" />
       <inertia
         ixx="5.83147818820347"
@@ -533,4 +543,9 @@
     <axis
       xyz="0 0 -1" />
+    <pid>
+      <p>1.0</p>
+      <i>0.1</i>
+      <d>0.01</d>
+    </pid>
   </joint>
   <link
@@ -541,5 +556,5 @@
         rpy="0 0 0" />
       <mass
-        value="0.317053240308613" />
+        value="3.17053240308613" />
       <inertia
         ixx="1.87953235728557"
@@ -586,4 +601,9 @@
     <axis
       xyz="0 0 1" />
+    <pid>
+      <p>1.0</p>
+      <i>0.1</i>
+      <d>0.01</d>
+    </pid>
   </joint>
   <link
@@ -594,5 +614,5 @@
         rpy="0 0 0" />
       <mass
-        value="0.291827459543752" />
+        value="2.91827459543752" />
       <inertia
         ixx="1.43479094583571"
@@ -639,4 +659,9 @@
     <axis
       xyz="0 0 -1" />
+    <pid>
+      <p>1.0</p>
+      <i>0.1</i>
+      <d>0.01</d>
+    </pid>
   </joint>
   <link
@@ -647,5 +672,5 @@
         rpy="0 0 0" />
       <mass
-        value="0.41227054564651" />
+        value="4.1227054564651" />
       <inertia
         ixx="1.92995623100548"
@@ -692,4 +717,9 @@
     <axis
       xyz="0 0 1" />
+    <pid>
+      <p>1.0</p>
+      <i>0.1</i>
+      <d>0.01</d>
+    </pid>
   </joint>
   <link
@@ -700,5 +730,5 @@
         rpy="0 0 0" />
       <mass
-        value="0.676402187018761" />
+        value="67.6402187018761" />
       <inertia
         ixx="7.05925773573284"
@@ -745,4 +775,9 @@
     <axis
       xyz="0 1 0" />
+    <pid>
+      <p>1.0</p>
+      <i>0.1</i>
+      <d>0.01</d>
+    </pid>
   </joint>
   <!-- <gazebo>
