Commit message: Manually moved joint locations to get things to export correctly

File: project_2/exports/aircraft_inspection_robot/urdf/aircraft_inspection_robot.urdf (robot description, URDF)
Before this commit: robot aircraft_inspection_robot, 14 links, 13 joints
Links:
- link arm_link_1: mass 25.9953851935799 -> 27.848718469127
- link back_right_wheel_link: mass 17.0942965183763 -> 17.0942965183762
- link camera_link: mass 67.6402186866665 -> 67.6402186866658
Joints:
- joint arm_link_1_joint: axis 1 0 0 -> 0 1 0; limit (none) -> lower=-1.57 upper=1.57 effort=100 velocity=1.57; origin xyz=0 0.3 0 rpy=0 0 0 -> xyz=-2.5994E-05 0.36854 0 rpy=0 0.083287 -1.5707; type continuous -> revolute
- joint arm_link_2_joint: limit (none) -> lower=-1.57 upper=1.57 effort=100 velocity=1.57; origin xyz=0 0.86 0 rpy=3.1416 0 3.1416 -> xyz=-0.83663 -0.0098939 -0.069842 rpy=0.083287 0 -1.5708; type continuous -> revolute
- joint arm_link_3_joint: limit (none) -> lower=-1.57 upper=1.57 effort=100 velocity=1.57; origin xyz=0 0.95 0 rpy=-3.1416 0 0 -> xyz=-0.010113 -0.91642 0 rpy=0 0 -1.6237E-05; type continuous -> revolute
- joint camera_holder_joint: origin xyz=0 -0.6096 0 rpy=-1.5708 0 -1.5708 -> xyz=-7.39773982035008E-05 -0.536820736088881 0 rpy=-1.57079640245877 0 -1.5709036865588
- joint rear_lidar_joint: origin xyz=-1.12750155043951 0.248338238939751 0.236097306217156 rpy=-1.57068141924114 0 3.14159265358979 -> xyz=-1.12750155043951 0.248337089864216 0.226097306283175 rpy=-1.57068141924114 0 3.14159265358979

Commit message: Added a whole bunch of points, axis, and origins to the solidworks model to make the axis of rotation and link origins generate correctly for the urdf exporter

File: project_2/exports/aircraft_inspection_robot/urdf/aircraft_inspection_robot.urdf (robot description, URDF)
Before this commit: robot aircraft_inspection_robot, 14 links, 13 joints
Links:
- removed link top_plate_link
- added link arm_connector_link, mass 2.62877306618386; collision mesh filename=package://aircraft_inspection_robot/meshes/arm_connector_li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; visual mesh filename=package://aircraft_inspection_robot/meshes/arm_connector_li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
- link arm_link_1: mass 27.848718469127 -> 27.8487184691269
- link arm_link_2: mass 22.8030311855106 -> 22.8030311855107
- link back_right_wheel_link: mass 17.0942965183762 -> 17.0942965183763
- link base_link: mass 16.3100062980245 -> 52.4458402259021
- link camera_link: mass 67.6402186866658 -> 67.6402186866665
Joints:
- removed joint top_plate_joint
- added joint arm_connect_joint: type fixed, parent base_link, child arm_connector_link, origin xyz=-0.4097 0.24836 0.41908 rpy=1.5707 0 0, axis 0 0 0
- joint arm_base_joint: origin xyz=0 0.01 0 rpy=3.14158139197888 1.57079625081358 3.14158139197905 -> xyz=0 0.05 0 rpy=3.14158142866165 1.57079625081358 3.14158142866183; parent top_plate_link -> arm_connector_link
- joint arm_link_1_joint: axis 0 1 0 -> 0 0 -1; limit lower=-1.57 upper=1.57 effort=100 velocity=1.57 -> lower=-1.57 upper=1.57 effort=10 velocity=1.57; origin xyz=-2.5994E-05 0.36854 0 rpy=0 0.083287 -1.5707 -> xyz=0 0.324649998991104 0 rpy=1.57079632679489 0 -1.57079632679575
- joint arm_link_2_joint: axis 1 0 0 -> 0 0 -1; limit lower=-1.57 upper=1.57 effort=100 velocity=1.57 -> lower=-1.57 upper=1.57 effort=10 velocity=1.57; origin xyz=-0.83663 -0.0098939 -0.069842 rpy=0.083287 0 -1.5708 -> xyz=-0.838219700899912 -7.9889090206009E-05 0 rpy=3.14159265358979 0 1.57079632018433
- joint arm_link_3_joint: axis 1 0 0 -> 0 0 -1; limit lower=-1.57 upper=1.57 effort=100 velocity=1.57 -> lower=-1.57 upper=1.57 effort=10 velocity=1.57; origin xyz=-0.010113 -0.91642 0 rpy=0 0 -1.6237E-05 -> xyz=7.9883045636886E-05 -0.914380299100637 0 rpy=0 -0.0773013935492111 -3.14158375334952
- joint back_left_wheel_joint: origin xyz=-0.70179757116575 0.534000833067587 0.101543460648476 rpy=-1.57057031157129 -1.03746333162058 3.14139810362434 -> xyz=-0.7018 0.534 0.10154 rpy=-1.5706 -1.0375 3.1414
- joint back_right_wheel_joint: origin xyz=-0.701797527934933 -0.0373531949241711 0.101609113542451 rpy=1.57061607230749 -0.879581000000789 0.000138956671881705 -> xyz=-0.7018 -0.037353 0.10161 rpy=1.5706 -0.87958 0.00013896
- joint camera_holder_joint: origin xyz=-7.39773982035008E-05 -0.536820736088881 0 rpy=-1.57079640245877 0 -1.5709036865588 -> xyz=0 0.537718005012817 0 rpy=-3.06429133570132 0 1.5707874531331
- joint camera_joint: origin xyz=0.152399998573732 0 0 rpy=0 0 0 -> xyz=0.152399998573742 0 0 rpy=0 0 0
- joint front_left_wheel_joint: origin xyz=-0.117597571165592 0.533998775516627 0.101543464746799 rpy=1.57061905476483 -0.865579426080518 0.00013506316993608 -> xyz=-0.117597571165592 0.533998775516627 0.101543464746798 rpy=1.57061905476483 -0.865579426080518 0.00013506316993608
- joint front_lidar_joint: origin xyz=0.30811 0.24834 0.2361 rpy=-1.5709 0 0 -> xyz=0.308106449560569 0.248338347564378 0.236097315694741 rpy=-1.57091123434865 0 0
- joint rear_lidar_joint: origin xyz=-1.12750155043951 0.248337089864216 0.226097306283175 rpy=-1.57068141924114 0 3.14159265358979 -> xyz=0.308106449560569 0.248338347564378 0.236097315694741 rpy=-1.57068141924114 0 3.14159265358979

Commit message: latest solidworks files

File: project_2/exports/aircraft_inspection_robot/urdf/aircraft_inspection_robot.urdf (robot description, URDF)
Before this commit: robot aircraft_inspection_robot, 14 links, 13 joints
Links:
- removed link arm_connector_link
- removed link camera_holder_link
- added link arm_link_4, mass 29.1827459543752; collision mesh filename=package://aircraft_inspection_robot/meshes/arm_link_4.STL; visual mesh filename=package://aircraft_inspection_robot/meshes/arm_link_4.STL
- added link arm_link_5, mass 41.227054564651; collision mesh filename=package://aircraft_inspection_robot/meshes/arm_link_5.STL; visual mesh filename=package://aircraft_inspection_robot/meshes/arm_link_5.STL
- link arm_base_link: mass 16.2102374081522 -> 49.4633477448353
- link arm_link_1: mass 27.8487184691269 -> 45.531535202482
- link arm_link_2: mass 22.8030311855107 -> 45.5315352024768
- link arm_link_3: mass 18.4583758499819 -> 31.7053240308613
- link back_left_wheel_link: mass 17.0942965183761 -> 26.0463122941313
- link back_right_wheel_link: mass 17.0942965183763 -> 26.0462008072991
- link base_link: mass 52.4458402259021 -> 52.3239752391313
- link camera_link: mass 67.6402186866665 -> 67.6402187018761
- link front_left_wheel_link: mass 17.0942965183763 -> 26.0463242126014
- link front_lidar_link: mass 21.0173459101461 -> 2.62716823876827
- link front_right_wheel_link: mass 17.0942965183764 -> 26.0461976105726
- link rear_lidar_link: mass 21.0173459127111 -> 2.62716823908889
Joints:
- removed joint arm_connect_joint
- removed joint camera_holder_joint
- removed joint camera_joint
- added joint arm_link_4_joint: type continuous, parent arm_link_3, child arm_link_4, origin xyz=-0.021323 -0.24407 0.508 rpy=-3.0713 -1.5708 1.4134, axis 0 0 -1
- added joint arm_link_5_joint: type continuous, parent arm_link_4, child arm_link_5, origin xyz=-0.127 0 -0.9234 rpy=1.5708 -0.087146 1.5708, axis 0 0 1
- added joint camera_link_joint: type fixed, parent arm_link_5, child camera_link, origin xyz=0.0121589249497853 0.139169858407754 -0.3556 rpy=3.05444641868214 -1.57079625379441 0, axis 0 0.999999993398127 0.00011490755350285
- joint arm_base_joint: origin xyz=0 0.05 0 rpy=3.14158142866165 1.57079625081358 3.14158142866183 -> xyz=-0.409742672306299 0.248387046108564 0.660376290839812 rpy=1.57079632680359 0.000114907553872355 1.57079640245869; parent arm_connector_link -> base_link
- joint arm_link_1_joint: limit lower=-1.57 upper=1.57 effort=10 velocity=1.57 -> (none); origin xyz=0 0.324649998991104 0 rpy=1.57079632679489 0 -1.57079632679575 -> xyz=0 0.266699994442256 -0.0254000017630377 rpy=-3.14159264700432 0 -3.05444635463409; type revolute -> continuous
- joint arm_link_2_joint: limit lower=-1.57 upper=1.57 effort=10 velocity=1.57 -> (none); origin xyz=-0.838219700899912 -7.9889090206009E-05 0 rpy=3.14159265358979 0 1.57079632018433 -> xyz=-0.069638 0.79706 0 rpy=-3.1416 0 0; type revolute -> continuous
- joint arm_link_3_joint: axis 0 0 -1 -> 0 0 1; limit lower=-1.57 upper=1.57 effort=10 velocity=1.57 -> (none); origin xyz=7.9883045636886E-05 -0.914380299100637 0 rpy=0 -0.0773013935492111 -3.14158375334952 -> xyz=-0.069638 -0.79706 0 rpy=0 0 0; type revolute -> continuous
- joint back_left_wheel_joint: axis 0 0 1 -> 0 0 0.999999999993264; origin xyz=-0.7018 0.534 0.10154 rpy=-1.5706 -1.0375 3.1414 -> xyz=-0.701797527935311 -0.0373482051170577 0.101609112969085 rpy=1.56727528936655 -1.5381898923507 0.00352290998991109
- joint back_right_wheel_joint: origin xyz=-0.7018 -0.037353 0.10161 rpy=1.5706 -0.87958 0.00013896 -> xyz=-0.701797527935311 -0.0373482051170577 0.101609112969085 rpy=1.57064724689163 -0.690734458596981 9.50549862212618E-05
- joint front_left_wheel_joint: origin xyz=-0.117597571165592 0.533998775516627 0.101543464746798 rpy=1.57061905476483 -0.865579426080518 0.00013506316993608 -> xyz=-0.117597527933808 -0.0373680425515616 0.10160911911045 rpy=1.57056878031369 -1.04143176730992 0.000196477434083904
- joint front_lidar_joint: origin xyz=0.308106449560569 0.248338347564378 0.236097315694741 rpy=-1.57091123434865 0 0 -> xyz=0.252189298222892 0.248326110601867 0.129347762825463 rpy=-1.57091123434865 0 0
- joint front_right_wheel_joint: axis 0 0 1 -> 0 0 0.999999999978938; origin xyz=-0.117597527934808 -0.0373548329643068 0.101609117592568 rpy=-1.57057710899586 -1.01905526588804 3.14140604048142 -> xyz=-0.117597527933808 -0.0373680425515616 0.10160911911045 rpy=-1.57068160265985 -0.0571716575997457 3.14159265358979
- joint rear_lidar_joint: origin xyz=0.308106449560569 0.248338347564378 0.236097315694741 rpy=-1.57068141924114 0 3.14159265358979 -> xyz=-1.07167463581468 0.248325943235427 0.129347754093208 rpy=-1.57068141924114 0 3.14159265358979
